File: KiCad/Antennenumschalter_V2.kicad_sch (KiCad schematic)
At the start: 40 parts, among them K1 LTV-816S, K2 LTV-816S, K3 LTV-816S, K4 LTV-816S, K5 7812, K6 LM1086-3.3, Q1 IRLML6401, Q2 IRLML6401, Q3 IRLML6401, Q4 IRLML6401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

Commit message: KiCad update
Parts:
- added H1, H2, H3, H4: MountingHole_Pad, MountingHole:MountingHole_3.2mm_M3_DIN965_Pad, symbol Mechanical:MountingHole_Pad
- K1, K2, K3, K4: value LTV-816S -> (none)
- S1: value RESET -> SW_MEC_5E
- X2: value ~ -> (none)
Connections:
- net GND: now also H1.1, H2.1, H3.1, H4.1
Other:
- company: (none) -> DM6RAC
- title: (none) -> WLAN-Antennenumschalter
- moved on the sheet: C1, C2, C3, C4, C5, C6, C7, C8, C9, F1, R1, R10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
